File: pcb/pr-clock.kicad_pcb (KiCad board)
At the start: 2 copper layers, 100 x 70 mm, 14 parts, among them J2 USB_C_Receptacle_USB2.0_14P, SW1 SW_Push, SW2 SW_Push, SW3 SW_Push, U1 TM1637, U2 ESP32-C3-WROOM-02, U3 ME6211C33M5

Commit message: add test firmware and bom
Parts:
- added J1: Conn_01x02, Connector_PinHeader_2.54mm:PinHeader_1x02_P2.54mm_Vertical, F.Cu at (190.8, 61.2)
Connections:
- U2 pad 11: unconnected-(U2-IO20/RXD-Pad11) -> Net-(J1-Pin_1)
- U2 pad 12: unconnected-(U2-IO21/TXD-Pad12) -> Net-(J1-Pin_2)
Routing:
- net Net-(J1-Pin_1): track 0.00 -> 16.3 mm, vias 0 -> 1
- net Net-(J1-Pin_2): track 0.00 -> 13.5 mm, vias 0 -> 1
- net GND: vias 33 -> 36
